File: CarHeadlightBuzzer/input.kicad_sch (KiCad schematic)
At the start: 5 parts, among them Q1 2N7000

Commit message: some routing
Parts:
- added R5 (x2): 5k, Resistor_THT:R_Axial_DIN0207_L6.3mm_D2.5mm_P2.54mm_Vertical, symbol Device:R
- added U3: LTV-817, Package_DIP:DIP-4_W7.62mm, symbol Isolator:LTV-817
Connections:
- net GND: now also U3.3
- net InputTTL: now also R5.2, U3.4; no longer Q1.3 (D)
- new net: Q1.3 (D), U3.2
- new net: R5.2, U3.1
- new net +5V: R5.1, R5.1
