File: CarHeadlightBuzzer/output.kicad_sch (KiCad schematic)
At the start: 7 parts, among them Q2 2N7000, Q3 IRF9Z34NPBF

Commit message: some routing
Parts:
- Z5: footprint DIOAD1068W53L380D172 -> SamacSys_Parts:DIOAD1068W53L380D172
Changed lines of the file:
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@@
       (effects (font (size 1.27 1.27)) (justify right))
     )
-    (property "Footprint" "DIOAD1068W53L380D172" (at 127 78.74 0)
+    (property "Footprint" "SamacSys_Parts:DIOAD1068W53L380D172" (at 127 78.74 0)
       (effects (font (size 1.27 1.27)) (justify left) hide)
     )
