File: CarHeadlightBuzzer/CarHeadlightBuzzer.kicad_sch (KiCad schematic)
At the start: 24 parts, among them IC1 LM2597MX-5.0_NOPB, J5 Conn_01x03, P1 Screw_Terminal_01x02, Q13 IRF9Z34NPBF, U1 ATmega328-P, U2 178.6165.0001, Y1 Crystal

Commit message: some routing
Parts:
- added J3: Conn_02x03_Odd_Even, Connector_PinHeader_2.54mm:PinHeader_2x03_P2.54mm_Vertical, symbol Connector_Generic:Conn_02x03_Odd_Even
- added J4: Conn_01x08, Connector_PinHeader_2.54mm:PinHeader_1x08_P2.54mm_Vertical, symbol Connector_Generic:Conn_01x08
- S1: footprint TS0266160BK260LCRD -> SamacSys_Parts:TS0266160BK260LCRD
- Y1: footprint (none) -> Crystal:Crystal_HC52-U_Vertical
Connections:
- net +5V: now also J3.2 (Pin_2)
- net GND: now also J3.6 (Pin_6)
- net LED: now also U1.13 (PD7); no longer U1.19 (PB5)
- net Output3: now also U1.15 (PB1); no longer U1.17 (PB3)
- net Reset: now also J3.5 (Pin_5)
- net D8: now reaches U1.14 (PB0)
- net D8: now also J4.1 (Pin_1)
- net D10: now reaches U1.16 (PB2)
- net D10: now also J4.2 (Pin_2)
- net MISO: now reaches U1.18 (PB4)
- net MISO: now also J3.1 (Pin_1)
- net A0: now reaches U1.23 (PC0)
- net A0: now also J4.3 (Pin_3)
- net A1: now reaches U1.24 (PC1)
- net A1: now also J4.4 (Pin_4)
- net A2: now reaches U1.25 (PC2)
- net A2: now also J4.5 (Pin_5)
- net A3: now reaches U1.26 (PC3)
- net A3: now also J4.6 (Pin_6)
- net A4: now reaches U1.27 (PC4)
- net A4: now also J4.7 (Pin_7)
- net A5: now reaches U1.28 (PC5)
- net A5: now also J4.8 (Pin_8)
- new net MOSI: J3.4 (Pin_4), U1.17 (PB3)
- new net SCK: J3.3 (Pin_3), U1.19 (PB5)
- no-connect marks 13 -> 2

Commit message: post routed and switched out the crystal needs to be inspected
Parts:
- Y1: footprint Crystal:Crystal_HC52-U_Vertical -> Crystal:Crystal_HC49-U_Vertical
Changed lines of the file:
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@@
       (effects (font (size 1.27 1.27)))
     )
-    (property "Footprint" "Crystal:Crystal_HC52-U_Vertical" (at 208.28 110.49 0)
+    (property "Footprint" "Crystal:Crystal_HC49-U_Vertical" (at 208.28 110.49 0)
       (effects (font (size 1.27 1.27)) hide)
     )
