File: CarHeadlightBuzzer/CarHeadlightBuzzer.kicad_pcb (KiCad board)
At the start: 2 copper layers, 59 parts, among them IC1 LM2597MX-5.0_NOPB, J1 Conn_01x03, J2 Conn_01x03, P1 Screw_Terminal_01x02, Q1 2N7000, Q10 IRF9Z34NPBF, Q2 2N7000, Q3 IRF9Z34NPBF, Q4 2N7000, Q5 2N7000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

Commit message: some routing
Parts:
- added J3: Conn_02x03_Odd_Even, Connector_PinHeader_2.54mm:PinHeader_2x03_P2.54mm_Vertical, F.Cu at (148.7, 88.5)
- added J4: Conn_01x08, Connector_PinHeader_2.54mm:PinHeader_1x08_P2.54mm_Vertical, F.Cu at (174.0, 103.7)
- added R20: 5k, Resistor_THT:R_Axial_DIN0207_L6.3mm_D2.5mm_P2.54mm_Vertical, F.Cu at (123.1, 71.2)
- added R21: 5k, Resistor_THT:R_Axial_DIN0207_L6.3mm_D2.5mm_P2.54mm_Vertical, F.Cu at (142.4, 71.3)
- added R22: 5k, Resistor_THT:R_Axial_DIN0207_L6.3mm_D2.5mm_P2.54mm_Vertical, F.Cu at (153.9, 52.9)
- added R23: 5k, Resistor_THT:R_Axial_DIN0207_L6.3mm_D2.5mm_P2.54mm_Vertical, F.Cu at (108.4, 71.3)
- added R24: 5k, Resistor_THT:R_Axial_DIN0207_L6.3mm_D2.5mm_P2.54mm_Vertical, F.Cu at (127.7, 71.4)
- added R25: 5k, Resistor_THT:R_Axial_DIN0207_L6.3mm_D2.5mm_P2.54mm_Vertical, F.Cu at (153.8, 67.9)
- added U3: LTV-817, Package_DIP:DIP-4_W7.62mm, F.Cu at (111.2, 68.9)
- added U4: LTV-817, Package_DIP:DIP-4_W7.62mm, F.Cu at (130.5, 69.0)
- added U5: LTV-817, Package_DIP:DIP-4_W7.62mm, F.Cu at (151.5, 64.8)
- added Y1: Crystal, Crystal:Crystal_HC52-U_Vertical, F.Cu at (154.6, 104.9)
- moved D1 118.5 mm to (107.8, 51.1)
- moved C1 118.0 mm to (107.7, 56.5)
- moved R1 117.8 mm to (116.3, 56.5)
- moved Q1 117.6 mm to (108.2, 62.8)
- moved R2 117.1 mm to (116.3, 62.5)
- moved Q7 113.2 mm to (112.2, 92.0), turned to -90 degrees
- moved D4 111.6 mm to (135.6, 51.1)
- moved C3 111.0 mm to (135.5, 56.5)
- moved R8 110.7 mm to (144.1, 56.5)
- moved Q5 110.4 mm to (136.1, 62.8)
- moved Z2 110.1 mm to (108.9, 100.1), turned to 90 degrees
- moved D3 109.7 mm to (121.9, 51.1)
- moved R9 109.6 mm to (144.1, 62.5)
- moved P1 109.4 mm to (99.3, 118.4), turned to -90 degrees
- moved C2 109.0 mm to (121.8, 56.5)
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Connections:
- Q1 pad 3: Input1 -> Net-(Q1-D)
- Q4 pad 3: Input2 -> Net-(Q4-D)
- Q5 pad 3: Input3 -> Net-(Q5-D)
- U1 pad 13: unconnected-(U1-PD7-Pad13) -> LED
- U1 pad 14: unconnected-(U1-PB0-Pad14) -> D8
- U1 pad 15: unconnected-(U1-PB1-Pad15) -> Output3
- U1 pad 16: unconnected-(U1-PB2-Pad16) -> D10
- U1 pad 17: Output3 -> MOSI
- U1 pad 18: unconnected-(U1-PB4-Pad18) -> MISO
- U1 pad 19: LED -> SCK
- U1 pad 23: unconnected-(U1-PC0-Pad23) -> A0
- U1 pad 24: unconnected-(U1-PC1-Pad24) -> A1
- U1 pad 25: unconnected-(U1-PC2-Pad25) -> A2
- U1 pad 26: unconnected-(U1-PC3-Pad26) -> A3
- U1 pad 27: unconnected-(U1-PC4-Pad27) -> A4
- U1 pad 28: unconnected-(U1-PC5-Pad28) -> A5
Routing:
- net GND: track 0.00 -> 389.5 mm
- net +VDC: track 0.00 -> 117.7 mm
- net +5V: track 0.00 -> 42.4 mm
- net Net-(Q8-Pad3): track 0.00 -> 19.3 mm
- net Net-(P1-Pin_1): track 0.00 -> 18.8 mm
- net Net-(IC1-DELAY): track 0.00 -> 18.1 mm
- net Net-(D6-K): track 0.00 -> 14.6 mm
- net /Output2/Output: track 0.00 -> 6.45 mm
- net Net-(IC1-ERROR_FLAG): track 0.00 -> 5.45 mm
- net Net-(Q10-Pad1): track 0.00 -> 4.72 mm
- net Net-(Q8-Pad1): track 0.00 -> 4.68 mm
- net Net-(IC1-~{SHUTDOWN}/SOFT-START): track 0.00 -> 3.99 mm
Other:
- board outline added: 88.9 x 104.1 mm

Commit message: post routed and switched out the crystal needs to be inspected
Parts:
- Y1: footprint Crystal:Crystal_HC52-U_Vertical -> Crystal:Crystal_HC49-U_Vertical
- moved C9 6.94 mm to (149.8, 116.5)
- moved C8 3.99 mm to (151.1, 100.1)
- moved Y1 2.80 mm to (151.9, 105.9)
Connections:
- R20 pad 2: unconnected-(R20-Pad2) -> Input1
- R21 pad 2: unconnected-(R21-Pad2) -> Input2
- R22 pad 2: unconnected-(R22-Pad2) -> Input3
- U3 pad 3: unconnected-(U3-Pad3) -> GND
- U3 pad 4: unconnected-(U3-Pad4) -> Input1
- U4 pad 3: unconnected-(U4-Pad3) -> GND
- U4 pad 4: unconnected-(U4-Pad4) -> Input2
- U5 pad 3: unconnected-(U5-Pad3) -> GND
- U5 pad 4: unconnected-(U5-Pad4) -> Input3
Routing:
- net +5V: track 42.4 -> 191.2 mm
- net Input1: track 0.00 -> 96.7 mm, vias 0 -> 1
- net MISO: track 0.00 -> 91.0 mm
- net GND: track 389.5 -> 455.6 mm
- net /Input2/Input: track 0.00 -> 56.8 mm
- net Input2: track 0.00 -> 55.7 mm
- net +VDC: track 117.7 -> 168.3 mm
- net Input3: track 0.00 -> 47.2 mm
- net Output1: track 0.00 -> 45.3 mm
- net /Input1/Input: track 0.00 -> 41.0 mm
- net Output3: track 0.00 -> 38.6 mm
- net LED: track 0.00 -> 35.9 mm
- net Output2: track 0.00 -> 35.2 mm
- net MOSI: track 0.00 -> 32.6 mm, vias 0 -> 1
- net RXttl: track 0.00 -> 31.9 mm
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Other:
- board text added: "+"
- board text added: "-"
- board text added: "2amp"
- board text added: "I1"
- board text added: "I2"
- board text added: "I3"
- board text added: "ISCP"
- board text added: "O1"
- board text added: "O2"
- board text added: "O3"

Commit message: last bits of stuff
Other:
- board text added: "Basic Bitch 328p Thingy V1.0"
- board text added: "RX"
- board text added: "TTL"
- board text added: "TX"
Changed lines of the file:
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@@
+    (effects (font (size 1.5 1.5) (thickness 0.3) bold) (justify left bottom))
+  )
+  (gr_text "TX" (at 176.146984 113.688311) (layer "F.SilkS")
+    (effects (font (size 1.5 1.5) (thickness 0.3) bold) (justify left bottom))
+  )
+  (gr_text "RX" (at 175.834368 111.17001) (layer "F.SilkS")
     (effects (font (size 1.5 1.5) (thickness 0.3) bold) (justify left bottom))
   )
@@
     (effects (font (size 1.5 1.5) (thickness 0.3) bold) (justify left bottom))
   )
+  (gr_text "TTL" (at 173.102228 119.620429) (layer "F.SilkS")
+    (effects (font (size 1.5 1.5) (thickness 0.3) bold) (justify left bottom))
+  )
   (gr_text "-" (at 91.951517 124.31911) (layer "F.SilkS")
     (effects (font (size 1.5 1.5) (thickness 0.3) bold) (justify left bottom))
@@
     (effects (font (size 1.5 1.5) (thickness 0.3) bold) (justify left bottom))
   )
+  (gr_text "Basic Bitch \n328p Thingy \nV1.0" (at 171.175468 133.08909) (layer "F.SilkS")
+    (effects (font (size 1.5 1.5) (thickness 0.3) bold))
+  )
   (gr_text "O2" (at 91.348265 92.036554) (layer "F.SilkS")
