File: BasicBitch328pThingy/input.kicad_sch (KiCad schematic)
At the start: 8 parts, among them Q1 2N7000, U3 LTV-817

Commit message: revamping this to have a CANBus Interface and swaping things to a SMD to save Space.
Parts:
- C2: footprint Capacitor_THT:C_Disc_D5.1mm_W3.2mm_P5.00mm -> Capacitor_SMD:C_1206_3216Metric_Pad1.33x1.80mm_HandSolder
- R1, R5: footprint Resistor_THT:R_Axial_DIN0207_L6.3mm_D2.5mm_P2.54mm_Vertical -> Resistor_SMD:R_1206_3216Metric_Pad1.30x1.75mm_HandSolder
