File: BasicBitch328pThingy/output.kicad_sch (KiCad schematic)
At the start: 7 parts, among them Q2 2N7000, Q3 IRF9Z34NPBF

Commit message: revamping this to have a CANBus Interface and swaping things to a SMD to save Space.
Parts:
- R6, R7, R8: footprint Resistor_THT:R_Axial_DIN0207_L6.3mm_D2.5mm_P2.54mm_Vertical -> Resistor_SMD:R_1206_3216Metric_Pad1.30x1.75mm_HandSolder
